File: PCB/PCB.kicad_sch (KiCad schematic)
At the start: 10 parts, among them J1_USB1 USB, J2A1 W5500_LEFT, J2B1 W5500_RIGHT, J3A1 PORTENTA_LEFT, J3B1 PORTENTA_RIGHT, J4A1 J_ESP32_LEFT, J4B1 J_ESP32_RIGHT, U1 AMS1117-3.3

Commit message: V5 PCB A Goeury
Parts:
- added C3: 100nF, Capacitor_SMD:C_0805_2012Metric, symbol Device:C
- added C4: 22uF, Capacitor_SMD:C_1206_3216Metric, symbol Device:C
- C1: value 10uF -> 22uF; footprint Package_TO_SOT_SMD:TO-252-2 -> Capacitor_SMD:C_1206_3216Metric
- C2: footprint Package_TO_SOT_SMD:TO-252-2 -> Capacitor_SMD:C_0805_2012Metric
Connections:
- net +3V3: now also C4.2
- net +5V_SYS: now also C3.2
- net GND: now also C3.1, C4.1
Other:
- moved on the sheet: C1, J1_USB1

Commit message: V8 Add ESP docs and PCB updates, adjust KiCad layout
Add ESP documentation (images + PDF) and an ESP32_PIN_MAPPING guide; include PCB fabrication PDFs and multiple PCB backups. Update KiCad project files (.kicad_pcb, .kicad_pro, .kicad_sch): reposition silkscreen labels, reassign ESP32 header nets, update pad/net mappings, modify many F.Cu segment coordinates and widths (widened traces), and refresh UUIDs to reflect rerouted layout. Also add esp/esp.ino and update esp/secrets.h and portenta/portenta.ino to match board changes and wiring.
Parts:
- C1, C2, C3, C4: KiLib_Generator (none) -> SMD_2terminal_chip_molded
- J1_USB1, J2A1, J2B1, J3A1, J3B1, J4A1, J4B1: KiLib_Generator (none) -> connector/pin_header_socket
Connections:
- net PORTENTA_RX: now also J4A1.7 (Pin_7); no longer J4A1.13 (Pin_13)
- net PORTENTA_TX: now also J4A1.6 (Pin_6); no longer J4A1.12 (Pin_12)
- net SPI_CS: now also J4A1.4 (Pin_4); no longer J4A1.8 (Pin_8)
- net W5500_INT: now also J4A1.3 (Pin_3); no longer J4A1.4 (Pin_4)
- net W5500_RST: now also J4A1.8 (Pin_8); no longer J4A1.5 (Pin_5)
Other:
- moved on the sheet: J4A1, J4B1
